File: coffee-scale.sch (KiCad schematic (older format))
At the start: 36 parts, among them IC1 esp8266-07, IC2 HX711, J1 Conn_01x04, J3 Conn_01x05_Male, J4 Conn_01x01_Male, J5 Conn_01x02, Q1 MMBT3906, SW1 SW_Push_JTP-1130, U1 LM1117-3.3

Commit message: next pcb version
fix esp position
add descriptions to copper
fix hole positions

Signed-off-by: Stefan Guelland <sguelland@thinkpad.za.w-hs.de>
Parts:
- added D2: LW_M673, Library:LW_M673, symbol Library:LW_M673
- added R10: 250, Resistor_SMD:R_0805_2012Metric_Pad1.15x1.40mm_HandSolder, symbol Device:R
- C10, C5: value 10u -> 1u
- J1: footprint Connector_Wire:SolderWirePad_1x04_P3.175mm_Drill0.8mm -> Connector_PinHeader_2.54mm:PinHeader_1x04_P2.54mm_Horizontal
Connections:
- net +3V3: now also R10.1
- net GND: now also J1.3 (Pin_3); no longer J1.2 (Pin_2)
- net LED: now reaches IC1.5 (GPIO14)
- net LED: now also D2.1 (K)
- net E+: now reaches C4.1, C5.1, IC2.3 (AVDD), Q1.3 (C), R3.1
- net E+: now also J1.4 (Pin_4); no longer J1.1 (Pin_1)
- net A-: now reaches R5.2
- net A-: now also J1.2 (Pin_2); no longer J1.3 (Pin_3)
- net A+: now reaches R6.1
- net A+: now also J1.1 (Pin_1); no longer J1.4 (Pin_4)
- new net: D2.2 (A), R10.2
Other:
- note added: "(3.3V - 2.8V) / 2mA = 250 Ohm"
Changed lines of the file:
@@
 Text GLabel 10400 3650 2    50   Input ~ 0
 RXD0
-Text GLabel 10400 3750 2    50   Input ~ 0
+Text GLabel 10400 3750 2    50   Output ~ 0
 TXD0
 $Comp
@@
 Text GLabel 10350 2100 2    50   Input ~ 0
 ~Bootloader
-Text GLabel 7200 1900 0    50   Input ~ 0
+Text GLabel 7200 1900 0    50   Output ~ 0
 ESP_ENABLE
 Text GLabel 9650 1700 2    50   Input ~ 0
@@
 P 3350 1650
 F 0 "C10" H 3465 1696 50  0000 L CNN
-F 1 "10u" H 3465 1605 50  0000 L CNN
+F 1 "1u" H 3465 1605 50  0000 L CNN
 F 2 "Capacitor_SMD:C_0805_2012Metric_Pad1.15x1.40mm_HandSolder" H 3388 1500 50  0001 C CNN
 F 3 "~" H 3350 1650 50  0001 C CNN
@@
 P 1650 2000
 F 0 "C5" H 1765 2046 50  0000 L CNN
-F 1 "10u" H 1765 1955 50  0000 L CNN
+F 1 "1u" H 1765 1955 50  0000 L CNN
 F 2 "Capacitor_SMD:C_0805_2012Metric_Pad1.15x1.40mm_HandSolder" H 1688 1850 50  0001 C CNN
 F 3 "~" H 1650 2000 50  0001 C CNN
@@
 L Connector_Generic:Conn_01x04 J1
 U 1 1 5C37632A
-P 750 2650
-F 0 "J1" H 670 2967 50  0000 C CNN
-F 1 "Conn_01x04" H 670 2876 50  0000 C CNN
-F 2 "Connector_Wire:SolderWirePad_1x04_P3.175mm_Drill0.8mm" H 750 2650 50  0001 C CNN
-F 3 "~" H 750 2650 50  0001 C CNN
-	1    750  2650
-	-1   0    0    -1
+P 750 2750
+F 0 "J1" H 670 3067 50  0000 C CNN
+F 1 "Conn_01x04" H 670 2976 50  0000 C CNN
+F 2 "Connector_PinHeader_2.54mm:PinHeader_1x04_P2.54mm_Horizontal" H 750 2750 50  0001 C CNN
+F 3 "~" H 750 2750 50  0001 C CNN
+	1    750  2750
+	-1   0    0    1
 $EndComp
 Wire Wire Line
@@
 Wire Wire Line
 	2300 5950 2550 5950
+Text Label 1300 1800 0    50   ~ 0
+E+
+Text Label 1450 2300 0    50   ~ 0
+E-
+$Comp
+L Device:R R10
+U 1 1 5C30450F
+P 8650 5600
+F 0 "R10" V 8443 5600 50  0000 C CNN
+F 1 "250" V 8534 5600 50  0000 C CNN
+F 2 "Resistor_SMD:R_0805_2012Metric_Pad1.15x1.40mm_HandSolder" V 8580 5600 50  0001 C CNN
+F 3 "~" H 8650 5600 50  0001 C CNN
+	1    8650 5600
+	0    1    1    0
+$EndComp
+Text Notes 8550 5950 0    50   ~ 0
+(3.3V - 2.8V) / 2mA = 250 Ohm
+$Comp
+L Library:LW_M673 D2
+U 1 1 5C314813
+P 8100 5600
+F 0 "D2" H 8091 5816 50  0000 C CNN
+F 1 "LW_M673" H 8091 5725 50  0000 C CNN
+F 2 "Library:LW_M673" H 8100 5350 50  0001 C CNN
+F 3 "~" H 8100 5700 50  0001 C CNN
+	1    8100 5600
+	1    0    0    -1
+$EndComp
+Text GLabel 7750 5600 0    50   Output ~ 0
+LED
+Wire Wire Line
+	7750 5600 7950 5600
+Wire Wire Line
+	8250 5600 8500 5600
+$Comp
+L power:+3.3V #PWR0111
+U 1 1 5C32CD9C
+P 8900 5500
+F 0 "#PWR0111" H 8900 5350 50  0001 C CNN
+F 1 "+3.3V" H 8915 5673 50  0000 C CNN
+F 2 "" H 8900 5500 50  0001 C CNN
+F 3 "" H 8900 5500 50  0001 C CNN
+	1    8900 5500
+	1    0    0    -1
+$EndComp
+Wire Wire Line
+	8900 5500 8900 5600
+Wire Wire Line
+	8900 5600 8800 5600
+Text GLabel 7500 2100 0    50   Input ~ 0
+LED
+Wire Wire Line
+	7700 2100 7500 2100
+Text Label 1800 3100 0    50   ~ 0
+A-
+Text Label 1800 3200 0    50   ~ 0
+A+
 $EndSCHEMATC
